File: e002_source/main.kicad_sch (KiCad schematic)
At the start: 28 parts, among them IC2 IC_TEXAS_TPS62743YFPR, IC3 IC_TEXAS_TPS62743YFPR, J3 USB_C_Receptacle_USB2.0_16P, U5 450mA 4.2V

Commit message: first commit of e002 rocker
Parts:
- removed C27: 10UF_0805_16V_X7R, smv_footprints:C_0805_2012Metric, symbol smv_capacitors:10UF_0805_16V_X7R
- removed C42: 4.7UF 0402 10V X7R, smv_footprints:C_0402_1005Metric, symbol smv_capacitors:4.7UF_0402_10V_X7R
- removed IC2: IC_TEXAS_TPS62743YFPR, smv_footprints:BGA8C40P2X4_87X156X53, symbol smv_ic:IC_TEXAS_TPS62743YFPR
- removed L2: 2.2u, smv_footprints:IND_MURATA_DFE201610P-2R2M=P2, symbol smv_inductors:IND_MURATA_DFE201610P-2R2M=P2
- removed L7: INDC_BEAD_BLM18AG601SN1D, Inductor_SMD:L_0603_1608Metric, symbol smv_inductors:INDC_BEAD_BLM18AG601SN1D
- added RV1, RV2, RV3: R_Potentiometer_MountingPin, Potentiometer_THT:Potentiometer_Vishay_148E-149E_Single_Horizontal, symbol Device:R_Potentiometer_MountingPin
Other:
- moved on the sheet: C43, C7, IC3, L3, L9
