File: e002_source/e002_rocker.kicad_sch (KiCad schematic)
At the start: 60 parts, among them IC1 IC_TEXAS_TPS62743YFPR, IC2 DRV8317HREER, J1 USB_C_Receptacle_USB2.0_16P, U1 ESP32-S3-WROOM-1-N8R2

Commit message: removed STM MCU to optimize cost
Parts:
- removed IC1: IC_TEXAS_TPS62743YFPR, smv_footprints:BGA8C40P2X4_87X156X53, symbol smv_ic:IC_TEXAS_TPS62743YFPR
- removed L2: 2.2u, smv_footprints:IND_MURATA_DFE201610P-2R2M=P2, symbol smv_inductors:IND_MURATA_DFE201610P-2R2M=P2
- added IC3: ~, smv_footprints:SOT95P280X125-6N, symbol smv_ic:IC_STM_DCP3601CDMR
- added J3: 5040500691, smv_footprints:CONN_MOLEX_5040500691, symbol smv_connectors_switches:CONN_MOLEX_5040500691
- added L3: INDC_TDK_VLCF5028T-220MR71-2, smv_footprints:IND_TDK_VLCF5028T-220MR71-2, symbol smv_inductors:INDC_TDK_VLCF5028T-220MR71-2
- added LED1, LED2: RGB, smv_footprints:DIOD_CREE_UHD111A-FKA-C3K23E1L3VG5ZB3Z3, symbol smv_diodes:DIOD_CREE_UHD111A-FKA-C3K23E1L3VG5ZB3Z3
- added MK1: ~, smv_footprints:IC_MIC_TDK_MMICT5837-00-012, symbol smv_ic:IC_MIC_TDK_MMICT5837-00-012
- added RV1: R_Potentiometer, Potentiometer_THT:Potentiometer_Alps_RK09L_Single_Vertical, symbol Device:R_Potentiometer
- added SW1, SW2: TS-1187A-B-A-B, ESWI-TL3342F160QG_V, symbol Altium Content Vault:root_3_SW-SPST-NO-4_Altium Content Vault
- added TP12: test point 1.5mm, TP1_FULL, symbol DAQ:root_0_Test Point_DAQ.SchLib
Connections:
- net +3V3: now also L3.2
- net ESP_EN: now also SW2.2
- net ESP_IO0: now also SW1.2, TP12.1
- net GND: now also IC2.21 (AGND), SW1.4, SW2.4
- net ISENS_A: now also C21.1, R16.1; no longer IC2.36 (SOA)
- net ISENS_B: now also C20.1, R14.1; no longer IC2.35 (SOB), R11.2, R14.2, R16.2
- net ISENS_C: now also C19.1, R11.1; no longer IC2.34 (SOC)
- net at C1.1, L1.2: now also IC3.5 (VIN)
- new net: IC3.6 (SW), L3.1
- new net: IC2.34 (SOC), R11.2
- new net: IC2.35 (SOB), R14.2
- new net: IC2.36 (SOA), R16.2
- now unconnected: U1.6 (IO6)
- no-connect marks 4 -> 11
Other:
- note added: "BOOT"
- note added: "ESP BOOT & RST buttons"
- note added: "RST"
- moved on the sheet: C10, C11, C12, C13, C14, C15, C16, C17, C19, C20, C21, C22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
