File: e003_source/e003_rocker.kicad_pcb (KiCad board)
At the start: 2 copper layers, 62 x 83 mm, 53 parts, among them J1 Conn_01x06_Pin, J2 Conn_02x05_Odd_Even, J3 Conn_01x04, J4 Conn_01x02_Pin, J5 SSQ-110-03-G-D, J6 SSQ-110-03-G-D, J7 Conn_02x05_Odd_Even, M1 CONN_M4_MOUNT, M2 CONN_M4_MOUNT, M3 CONN_M4_MOUNT, M4 CONN_M4_MOUNT, M5 CONN_M4_MOUNT, SW1 BTN_OMRON_B3S-1100P, SW3 BTN_OMRON_B3S-1100P, U1 ESP32-S3-WROOM-1-N8R2

Commit message: before real start of EVT
Routing:
- net GND: track 32.6 -> 34.4 mm
Changed lines of the file:
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@@
 			(drillshape 0)
 			(scaleselection 1)
-			(outputdirectory "")
+			(outputdirectory "gerber/")
 		)
 	)
@@
 			)
 			(layer "B.SilkS")
-			(net 7798903)
 		)
 		(fp_line
@@
 			)
 			(layer "B.SilkS")
-			(net 7798903)
 		)
 		(fp_line
@@
 			)
 			(layer "B.SilkS")
-			(net 7798903)
 		)
 		(fp_line
@@
 			)
 			(layer "B.SilkS")
-			(net 7798903)
 		)
 		(fp_rect
@@
 			(fill yes)
 			(layer "B.SilkS")
-			(net 7798903)
 		)
 		(fp_line
@@
 			)
 			(layer "User.6")
-			(net 7798903)
 		)
 		(fp_line
@@
 			)
 			(layer "User.6")
-			(net 7798903)
 		)
 		(fp_line
@@
 			)
 			(layer "User.6")
-			(net 7798903)
 		)
 		(fp_line
@@
 			)
 			(layer "User.6")
-			(net 7798903)
 		)
 		(fp_text user "${REFERENCE}"
@@
 		)
 		(embedded_fonts no)
-		(embedded_files)
 		(model "kicad-embed://SSQ-110-03-T-D.stp"
 			(offset
@@
 			)
 			(layer "B.SilkS")
-			(net 7798903)
 		)
 		(fp_line
@@
 			)
 			(layer "B.SilkS")
-			(net 7798903)
 		)
 		(fp_line
@@
 			)
 			(layer "B.SilkS")
-			(net 7798903)
 		)
 		(fp_line
@@
 			)
 			(layer "B.SilkS")
-			(net 7798903)
 		)
 		(fp_rect
@@
 			(fill yes)
 			(layer "B.SilkS")
-			(net 7798903)
 		)
 		(fp_line
@@
 			)
 			(layer "User.6")
-			(net 7798903)
 		)
 		(fp_line
@@
 			)
 			(layer "User.6")
-			(net 7798903)
 		)
 		(fp_line
@@
 			)
 			(layer "User.6")
-			(net 7798903)
 		)
 		(fp_line
@@
 			)
 			(layer "User.6")
-			(net 7798903)
 		)
 		(fp_text user "${REFERENCE}"
@@
 		)
 		(embedded_fonts no)
-		(embedded_files)
 		(model "kicad-embed://SSQ-110-03-T-D.stp"
 			(offset
@@
 	)
 	(segment
+		(start 123 168)
+		(end 123 167.4)
+		(width 0.2)
+		(layer "F.Cu")
+		(net 1)
+	)
+	(segment
 		(start 119.75 150.4)
 		(end 119.75 150.275)
@@
 	)
 	(segment
+		(start 123 167.4)
+		(end 123.8 166.6)
+		(width 0.2)
+		(layer "F.Cu")
+		(net 1)
+	)
+	(segment
 		(start 141.875 115.5)
 		(end 141.875 116.85)
@@
 	)
 	(embedded_fonts no)
-	(embedded_files)
 )
