File: e003_source/e003_rocker.kicad_sch (KiCad schematic)
At the start: 53 parts, among them J1 Conn_01x06_Pin, J2 Conn_02x05_Odd_Even, J3 Conn_01x04, J4 Conn_01x02_Pin, J5 SSQ-110-03-G-D, J6 SSQ-110-03-G-D, J7 Conn_02x05_Odd_Even, M1 CONN_M4_MOUNT, M2 CONN_M4_MOUNT, M3 CONN_M4_MOUNT, M4 CONN_M4_MOUNT, M5 CONN_M4_MOUNT, SW1 BTN_OMRON_B3S-1100P, SW3 BTN_OMRON_B3S-1100P, U1 ESP32-S3-WROOM-1-N8R2

Commit message: before real start of EVT
Parts:
- removed C1: CL10A105KB8NNNC, Capacitor_SMD:C_0603_1608Metric_Pad1.08x0.95mm_HandSolder, symbol Altium Content Vault:root_0_b4654b650e69147ec39a6b967a45e02_Altium Content Vault
- removed C3, C4, C5: 100NF_0201_10V_X7R, smv_footprints:C_0603_1608Metric, symbol smv_capacitors:100NF 0603 50V X7R
- removed J5, J6: SSQ-110-03-G-D, Vault:Samtec_SSQ-110-03-x-D, symbol Altium Vault - TI:root_0_mirrored_Receptacle_10x2_Altium Vault - TI
- removed RV1, RV2, RV3: R_Potentiometer, Potentiometer_THT:Potentiometer_Alpha_RD901F-40-00D_Single_Vertical, symbol Device:R_Potentiometer
- added C1, C13: CAPP_PANASONIC_EEV-FK1E222M, smv_footprints:CAPP_PANASONIC_EEEFK0J682AM, symbol smv_capacitors:CAPP_PANASONIC_EEV-FK1E222M
- added C14, C15, C16, C17, C19, C20: 10UF_1206_35V_X5R, smv_footprints:C_1206_3216Metric, symbol smv_capacitors:10UF_1206_35V_X5R
- added C22, C26, C27: 100NF 0402 25V X7R, smv_footprints:C_0402_1005Metric, symbol smv_capacitors:100NF 0402 25V X7R
- added C28: 1UF 0603 16V X7R, smv_footprints:C_0603_1608Metric, symbol smv_capacitors:1UF 0603 16V X7R
- added C29: 4.7NF 0603 100V X7R, smv_footprints:C_0603_1608Metric, symbol smv_capacitors:47NF_0603_25V_X7R
- added C3, C4, C5: 4.7NF 0603 100V X7R, smv_footprints:C_0603_1608Metric, symbol smv_capacitors:4.7NF_0603_50V_X7R
- added C30: 2.2UF 0402 16V X5R, smv_footprints:C_0402_1005Metric, symbol smv_capacitors:2.2UF_0402_16V_X5R
- added C31: 4.7UF 0402 10V X7R, smv_footprints:C_0402_1005Metric, symbol smv_capacitors:4.7UF_0402_10V_X7R
- added C32: 10UF_0805_16V_X7R, smv_footprints:C_0805_2012Metric, symbol smv_capacitors:10UF_0805_16V_X7R
- added IC1: DRV8317HREER, smv_footprints:QFN40P400X500X80-37N-D, symbol DRV8317HREER:DRV8317HREER
- added IC3: ~, smv_footprints:SOT95P280X125-6N, symbol smv_ic:IC_STM_DCP3601CDMR
- added L1: INDC_BEAD_BLM18AG601SN1D, Inductor_SMD:L_0603_1608Metric, symbol smv_inductors:INDC_BEAD_BLM18AG601SN1D
- added L3: INDC_TDK_VLCF5028T-220MR71-2, smv_footprints:IND_TDK_VLCF5028T-220MR71-2, symbol smv_inductors:INDC_TDK_VLCF5028T-220MR71-2
- added R19, R20, R21, R22, R23, R24: 0R 0603, smv_footprints:R_0603_1608Metric, symbol smv_resistors:0R 0603
- added R25, R26, R28: 10R 0402, smv_footprints:R_0402_1005Metric, symbol smv_resistors:10R 0402
- added R27: 10K 0603, smv_footprints:R_0603_1608Metric, symbol smv_resistors:10K 0603
- added U2: RS2254XQ, smv_footprints:IC_RUNIC_RS2254XQ, symbol smv_ic:IC_RUNIC_RS2254
- R14, R15, R16: symbol smv_resistors:100R 0603 -> smv_resistors:1K 0603; val 100R -> 1k
Connections:
- net +3V3: now also C32.1, L3.2, R19.2, R21.2, R23.2, R27.2
- net DRV-INHA: now also IC1.23 (INHA)
- net DRV-INHB: now also IC1.25 (INHB)
- net DRV-INHC: now also IC1.27 (INHC)
- net GIO10: no longer U1.18 (IO10)
- net GND: now also C1.2 (-), C13.2 (-), C14.2, C15.2, C16.2, C17.2, C19.2, C20.2, C22.2, C26.2, C27.2, C3.2, C30.2, C31.2, C32.2, C4.2, C5.2, IC1.10 (PGND_1), IC1.13 (PGND_2), IC1.16 (PGND_3), IC1.19 (PGND_4), IC1.21 (AGND), IC1.37 (GND), R20.1, R22.1, R24.1, U2.7 (VSS)
- new net: C22.1, IC1.33 (CSAREF)
- new net: C31.1, IC3.5 (VIN), L1.2
- new net: IC3.6 (SW), L3.1
- new net: IC1.2 (NFAULT), R27.1
- new net: C1.1 (+), C13.1 (+), C14.1, C15.1, C16.1, C17.1, C19.1, C20.1, C26.1, C27.1, C28.1, IC1.20 (VM_3), IC1.7 (VIN_AVDD), IC1.8 (VM_1), IC1.9 (VM_2)
- new net: IC1.29 (GAIN), R19.1, R20.2
- new net: IC1.30 (SLEW), R21.1, R22.2
- new net: IC1.31 (MODE), R23.1, R24.2
- new net: IC1.34 (SOC), R28.2
- new net: IC1.35 (SOB), R26.2
- new net: IC1.36 (SOA), R25.2
- new net: C29.2, IC1.4 (CPL)
- new net: C29.1, IC1.5 (CPH)
- new net: C28.2, IC1.6 (CP)
- new net: C5.1, U2.9 (SIG_C_OUT_IN)
- new net: R28.1, U2.8 (SIG_C_IN_OUT)
- new net: R25.1, U2.1 (SIG_A_IN_OUT)
- new net: C3.1, U2.2 (SIG_A_OUT_IN)
- new net: C4.1, U2.3 (SIG_B_OUT_IN)
- new net: R26.1, U2.4 (SIG_B_IN_OUT)
- new net +BATT: L1.1
- new net DRV_AVDD: C30.1, IC1.22 (AVDD)
- new net MOTOR_A: IC1.11 (OUTA_1), IC1.12 (OUTA_2)
- new net MOTOR_B: IC1.14 (OUTB_1), IC1.15 (OUTB_2)
- new net MOTOR_C: IC1.17 (OUTC_1), IC1.18 (OUTC_2)
- new net SAMPLE_HOLD: U1.18 (IO10), U2.12 (CONTROL_D), U2.13 (CONTROL_A), U2.5 (CONTROL_B), U2.6 (CONTROL_C)
- no-connect marks 25 -> 12
Other:
- note removed: "For internal use only"
- note removed: "LAUNCHPAD CONNECTIONS"
- note removed: "Mates with J1/J3 on Launchpad"
- note removed: "Mates with Launchpad J4/J2"
- note removed: "R2/R48 DNP"
- note removed: "R51 DNP"
- note removed: "To be used with LAUNCHXL-F280049C headers J1/J3 and J4/J2"
- moved on the sheet: J1, J2, J4, M1, M2, M3, M4, M5, R1, R2, R4, R5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

Commit message: first evt to jlc
Parts:
- removed C1, C13: CAPP_PANASONIC_EEV-FK1E222M, smv_footprints:CAPP_PANASONIC_EEEFK0J682AM, symbol smv_capacitors:CAPP_PANASONIC_EEV-FK1E222M
- removed C14, C15, C16, C17, C19, C20: 10UF_1206_35V_X5R, smv_footprints:C_1206_3216Metric, symbol smv_capacitors:10UF_1206_35V_X5R
- removed C22, C26, C27: 100NF 0402 25V X7R, smv_footprints:C_0402_1005Metric, symbol smv_capacitors:100NF 0402 25V X7R
- removed C28: 1UF 0603 16V X7R, smv_footprints:C_0603_1608Metric, symbol smv_capacitors:1UF 0603 16V X7R
- removed C29: 4.7NF 0603 100V X7R, smv_footprints:C_0603_1608Metric, symbol smv_capacitors:47NF_0603_25V_X7R
- removed C3, C4, C5: 4.7NF 0603 100V X7R, smv_footprints:C_0603_1608Metric, symbol smv_capacitors:4.7NF_0603_50V_X7R
- removed C30: 2.2UF 0402 16V X5R, smv_footprints:C_0402_1005Metric, symbol smv_capacitors:2.2UF_0402_16V_X5R
- removed C7, C8, C9: 220PF 0603 50V C0G, smv_footprints:C_0603_1608Metric, symbol smv_capacitors:220PF 0603 50V C0G
- removed IC1: DRV8317HREER, smv_footprints:QFN40P400X500X80-37N-D, symbol DRV8317HREER:DRV8317HREER
- removed J2: Conn_02x05_Odd_Even, Connector_PinHeader_2.00mm:PinHeader_2x05_P2.00mm_Vertical, symbol Connector_Generic:Conn_02x05_Odd_Even
- removed J3: Conn_01x04, Connector_PinHeader_2.54mm:PinHeader_1x04_P2.54mm_Horizontal, symbol Connector_Generic:Conn_01x04
- removed J7: Conn_02x05_Odd_Even, Connector_PinHeader_2.54mm:PinHeader_2x05_P2.54mm_Vertical, symbol Connector_Generic:Conn_02x05_Odd_Even
- removed M3: CONN_M4_MOUNT, MountingHole:MountingHole_2.7mm_M2.5_ISO7380_Pad, symbol smv_connectors_switches:CONN_M4_MOUNT
- removed R1, R2, R4, R5, R6: 1K 0603, smv_footprints:R_0603_1608Metric, symbol smv_resistors:1K 0603
- removed R10, R11, R9: 100R 0603, smv_footprints:R_0603_1608Metric, symbol smv_resistors:100R 0603
- removed R12, R27: 10K 0603, smv_footprints:R_0603_1608Metric, symbol smv_resistors:10K 0603
- removed R13: 100K 0603, smv_footprints:R_0603_1608Metric, symbol smv_resistors:100K 0603
- removed R14, R15, R16: 100R 0603, smv_footprints:R_0603_1608Metric, symbol smv_resistors:1K 0603
- removed R17: 5.6K 0603, smv_footprints:R_0603_1608Metric, symbol smv_resistors:5.6K 0603
- removed R19, R20, R21, R22, R23, R24: 0R 0603, smv_footprints:R_0603_1608Metric, symbol smv_resistors:0R 0603
- removed R25, R26, R28: 10R 0402, smv_footprints:R_0402_1005Metric, symbol smv_resistors:10R 0402
- removed U2: RS2254XQ, smv_footprints:IC_RUNIC_RS2254XQ, symbol smv_ic:IC_RUNIC_RS2254
- added C1, C12, C19, C2, C20, C44, C46, C5, C56, C57, C59, C6, C7, C9: 100NF 0402 25V X7R, smv_footprints:C_0402_1005Metric, symbol smv_capacitors:100NF 0402 25V X7R
- added C13, C14: 10UF_0805_16V_X7R, smv_footprints:C_0805_2012Metric, symbol smv_capacitors:10UF_0805_16V_X7R
- added C15: 100NF 1206 50V C0G, smv_footprints:C_1206_3216Metric, symbol smv_capacitors:100NF_1206_50V_C0G
- added C24, C28, C29: 220PF 0603 50V C0G, smv_footprints:C_0603_1608Metric, symbol smv_capacitors:220PF 0603 50V C0G
- added C4: 4.7N 50 VDC 5% 0603 C0G, smv_footprints:C_0603_1608Metric, symbol smv_capacitors:4.7NF_0603_50V_C0G
- added C41, C58, C62, C8: 100NF_0603_100V_X7S, smv_footprints:C_0603_1608Metric, symbol smv_capacitors:100NF_0603_100V_X7S
- added D1: DOID_ST_ESDA25P35-1U1M, smv_footprints:DIOD_STM_ESDA25P35-1U1M, symbol smv_diodes:DOID_ST_ESDA25P35-1U1M
- added D9: DIODE_DIODES_B260S1F-7, smv_footprints:D_SOD-123F, symbol smv_diodes:DIODE_DIODES_B260S1F-7
- added F1: 2A 3.5A 16V, smv_footprints:PFUSE_LITTLEFUSE_1812L20016DR, symbol smv_resistors:PFUSE_LITTLEFUSE_1812L20016DR
- added IC1: IC_DIODES_AP7381-50Y-13, smv_footprints:IC_DIODES_AP738133Y13, symbol smv_ic:IC_DIODES_AP7381-50Y-13
- added IC5: IC_DIODES_AP7381-33Y-13, smv_footprints:IC_DIODES_AP738133Y13, symbol smv_ic:IC_DIODES_AP7381-33Y-13
- added J1: CONN_GCT_USB4105-GF-A, Connector_USB:USB_C_Receptacle_GCT_USB4105-xx-A_16P_TopMnt_Horizontal, symbol smv_connectors_switches:CONN_GCT_USB4105-GF-A
- added J9: CONN_AMPHENOL_F51L-1A7H1-11018, smv_footprints:CONN_AMPHENOL_F51L-1A7H1-11018, symbol smv_connectors_switches:CONN_AMPHENOL_F51L-1A7H1-11018
- added L13, L20, L21, L22, L23, L25, L6, L7, L8, L9: INDC_BEAD_BLM18AG601SN1D, Inductor_SMD:L_0603_1608Metric, symbol smv_inductors:INDC_BEAD_BLM18AG601SN1D
- added L3: INDC_BEAD_TAY_FBMH3216HM221NT, smv_footprints:INDC_TAY_FBMH3216HM221NT, symbol smv_inductors:INDC_BEAD_TAY_FBMH3216HM221NT
- added M11, M12, M13: CONN_M4_MOUNT, MountingHole:MountingHole_2.7mm_M2.5_ISO7380_Pad, symbol smv_connectors_switches:CONN_M4_MOUNT
- added MK2: IC_KNOWLES_SPH0141LM4H-1, smv_footprints:MIC_KNOWLES_SPH0641LM4H-1, symbol smv_ic:IC_KNOWLES_SPH0141LM4H-1
- added Q1, Q5: TRAN_ALPHA_AONR21357, smv_footprints:TRAN_ALPHA__AONR21307, symbol smv_transistors:TRAN_ALPHA_AONR21357
- added R1: 220K 0402, smv_footprints:R_0402_1005Metric, symbol smv_resistors:220K 0402
- added R10, R22, R56, R59, R61, R62, R7: 100R 0402, smv_footprints:R_0402_1005Metric, symbol smv_resistors:100R 0402
- added R11, R30, R32, R33, R50, R58, R60, R72: 47K 0402, smv_footprints:R_0402_1005Metric, symbol smv_resistors:47K 0402
- added R12, R21, R6, R8, R9: 4.7K 0402, smv_footprints:R_0402_1005Metric, symbol smv_resistors:4.7K 0402
- added R14, R15, R17, R5, R53, R54: 1.5K 0402, smv_footprints:R_0402_1005Metric, symbol smv_resistors:1.5K 0402
- added R2: 80.6K 0402 1%, smv_footprints:R_0402_1005Metric, symbol smv_resistors:80.6K_0402
- added R3: 28K 0402 1%, smv_footprints:R_0402_1005Metric, symbol smv_resistors:28K 0402
- added R49, R51, R55: 10R 0402, smv_footprints:R_0402_1005Metric, symbol smv_resistors:10R 0402
- added R52, R73: 10K 0402, smv_footprints:R_0402_1005Metric, symbol smv_resistors:10K 0402
- added R57: 7.5K 0402, smv_footprints:R_0402_1005Metric, symbol smv_resistors:7.5K_0402
- added TP1, TP13, TP2, TP3: TestPoint, smv_footprints:TestPoint_Loop_D2.60mm_Drill1.4mm_Beaded, symbol smv_connectors_switches:TestPoint_2_6mm_Beaded
- added U1: IC_TEXAS_TPD4S201TRGRRQ1, smv_footprints:IC_TEXAS_TPD4S201TRGR, symbol smv_ic:IC_TEXAS_TPD4S201TRGRRQ1
- added U2: HUSB238_002DD, Package_DFN_QFN:DFN-10-1EP_3x3mm_P0.5mm_EP1.65x2.38mm, symbol smv_ic:IC_HYNETEK_HUSB238
- C11: renamed from C25; value 100NF_0201_10V_X7R -> 100NF 1206 50V C0G; symbol smv_capacitors:100NF 0603 50V X7R -> smv_capacitors:100NF_1206_50V_C0G; Voltage 0V -> (none); manfn# Generic -> (none); val 100nF -> 100N
- C16: renamed from C2; value 100NF_0201_10V_X7R -> 100NF 0402 25V X7R; footprint smv_footprints:C_0603_1608Metric -> smv_footprints:C_0402_1005Metric; symbol smv_capacitors:100NF 0603 50V X7R -> smv_capacitors:100NF 0402 25V X7R; Voltage 0V -> (none); manfn# Generic -> (none)
- C18: value 1UF 0603 16V X7R -> 100NF 0402 25V X7R; footprint smv_footprints:C_0603_1608Metric -> smv_footprints:C_0402_1005Metric; symbol smv_capacitors:1UF 0603 16V X7R -> smv_capacitors:100NF 0402 25V X7R; Voltage 0V -> (none); manfn# Generic -> (none); val 1uF -> 100nF
- C21: renamed from C12; Voltage 0V -> (none); manfn# Generic -> (none)
- C22: renamed from C11; Voltage 0V -> (none); manfn# Generic -> (none)
- C23: renamed from C10; Voltage 0V -> (none); manfn# Generic -> (none)
- C25: renamed from C6; value 1UF 0603 16V X7R -> 100NF 0402 25V X7R; footprint smv_footprints:C_0603_1608Metric -> smv_footprints:C_0402_1005Metric; symbol smv_capacitors:1UF 0603 16V X7R -> smv_capacitors:100NF 0402 25V X7R; ALTIUM_VALUE 1uF -> (none); AUTOMOTIVE No -> (none); CAPACITANCE 1uF -> (none); CATEGORY Cap -> (none); COMPONENTLINK2DESCRIPTION Datasheet -> (none); COMPONENTLINK2URL http://www.samsungsem.com/global/front/downloadcms.do?path=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 -> (none); DEVICE CLASS L1 Passive Components -> (none); DEVICE CLASS L2 Capacitors -> (none); DEVICE CLASS L3 Ceramic Capacitors -> (none); DIGIKEY DESCRIPTION CAP CER 1UF 16V X7R 0603 -> (none); HEIGHT 0.9mm -> (none); IPC LAND PATTERN NAME CAPC16080X80 -> (none); LCSC C15849 -> (none); LEAD FREE Yes -> (none); MANUFACTURER Samsung Electro-Mechanics America, Inc -> (none); MANUFACTURER PART NUMBER CL10B105KO8NNNC -> (none); MATERIAL Ceramic -> (none); OCTOPART https://octopart.com/cl10b105ko8nnnc-samsung-19018973 -> (none); PACKAGE CL10B105KO8NNNC -> (none); ROHS TRUE -> (none); TEMPERATURE -55°C to +125°C -> (none); TEMPERATURE CHARACTERISTIC X5R -> (none); TEMPERATURE COEFFICIENT 15% -> (none); TEMPERATURE RANGE HIGH +125°C -> (none); TEMPERATURE RANGE LOW -55°C -> (none); TOLERANCE 10% -> (none); VOLTAGE RATING 50V -> (none); Voltage 0V -> (none); manfn# Generic -> (none); val 1uF -> 100nF
- C26: renamed from C23; value 10UF_1206_35V_X5R -> 10UF_0805_16V_X7R; footprint smv_footprints:C_1206_3216Metric -> smv_footprints:C_0805_2012Metric; symbol smv_capacitors:10UF_1206_35V_X5R -> smv_capacitors:10UF_0805_16V_X7R; CAPACITANCE 22uF -> (none); CASE CODE (IMPERIAL) 1206 -> (none); CASE CODE (METRIC) 3216 -> (none); CASE/PACKAGE 1206 -> (none); DEPTH 1.6mm -> (none); DIELECTRIC X5R -> (none); HEIGHT 1.6mm -> (none); LCSC C5672 -> (none); LEAD FREE Lead Free -> (none); LENGTH 3.2mm -> (none); MAX OPERATING TEMPERATURE 85°C -> (none); MIN OPERATING TEMPERATURE -55°C -> (none); MOUNT Surface Mount -> (none); PACKAGE QUANTITY 1 -> (none); PACKAGING Tape and Reel -> (none); RADIATION HARDENING No -> (none); THICKNESS 0.071inch -> (none); TOLERANCE 10% -> (none); VOLTAGE RATING 10V -> (none); VOLTAGE RATING (DC) 10V -> (none); Voltage 0V -> (none); WIDTH 0.063inch -> (none); manfn# Generic -> (none)
- C27: renamed from C24; value 1UF 0603 16V X7R -> 100NF 0402 25V X7R; footprint smv_footprints:C_0603_1608Metric -> smv_footprints:C_0402_1005Metric; symbol smv_capacitors:1UF 0603 16V X7R -> smv_capacitors:100NF 0402 25V X7R; ALTIUM_VALUE 1uF -> (none); AUTOMOTIVE No -> (none); CAPACITANCE 1uF -> (none); CATEGORY Cap -> (none); COMPONENTLINK2DESCRIPTION Datasheet -> (none); COMPONENTLINK2URL http://www.samsungsem.com/global/front/downloadcms.do?path=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 -> (none); DEVICE CLASS L1 Passive Components -> (none); DEVICE CLASS L2 Capacitors -> (none); DEVICE CLASS L3 Ceramic Capacitors -> (none); DIGIKEY DESCRIPTION CAP CER 1UF 16V X7R 0603 -> (none); HEIGHT 0.9mm -> (none); IPC LAND PATTERN NAME CAPC16080X80 -> (none); LCSC C15849 -> (none); LEAD FREE Yes -> (none); MANUFACTURER Samsung Electro-Mechanics America, Inc -> (none); MANUFACTURER PART NUMBER CL10B105KO8NNNC -> (none); MATERIAL Ceramic -> (none); OCTOPART https://octopart.com/cl10b105ko8nnnc-samsung-19018973 -> (none); PACKAGE CL10B105KO8NNNC -> (none); ROHS TRUE -> (none); TEMPERATURE -55°C to +125°C -> (none); TEMPERATURE CHARACTERISTIC X5R -> (none); TEMPERATURE COEFFICIENT 15% -> (none); TEMPERATURE RANGE HIGH +125°C -> (none); TEMPERATURE RANGE LOW -55°C -> (none); TOLERANCE 10% -> (none); VOLTAGE RATING 50V -> (none); Voltage 0V -> (none); manfn# Generic -> (none); val 1uF -> 100nF
- C3: renamed from C31; value 4.7UF 0402 10V X7R -> 100NF 0402 25V X7R; symbol smv_capacitors:4.7UF_0402_10V_X7R -> smv_capacitors:100NF 0402 25V X7R; Voltage 0V -> (none); manfn# Generic -> (none); val 4.7uF -> 100nF
- IC2: renamed from IC3; value ~ -> DCP3601
- J3: renamed from J1; footprint Connector_PinHeader_2.54mm:PinHeader_1x06_P2.54mm_Vertical -> (none)
- J4: footprint TerminalBlock:TerminalBlock_Xinya_XY308-2.54-2P_1x02_P2.54mm_Horizontal -> (none)
- M1, M2, M4, M5: now in the parts list
- R16: renamed from R8; value 100R 0603 -> 100R 0402; footprint smv_footprints:R_0603_1608Metric -> smv_footprints:R_0402_1005Metric; symbol smv_resistors:100R 0603 -> smv_resistors:100R 0402
- R18: renamed from R7; value 100R 0603 -> 100R 0402; footprint smv_footprints:R_0603_1608Metric -> smv_footprints:R_0402_1005Metric; symbol smv_resistors:100R 0603 -> smv_resistors:100R 0402
- R19: renamed from R3; value 100R 0603 -> 100R 0402; footprint smv_footprints:R_0603_1608Metric -> smv_footprints:R_0402_1005Metric; symbol smv_resistors:100R 0603 -> smv_resistors:100R 0402
- R20: renamed from R18; value 10K 0603 -> 10K 0402; footprint smv_footprints:R_0603_1608Metric -> smv_footprints:R_0402_1005Metric; symbol smv_resistors:10K 0603 -> smv_resistors:10K 0402
- renumbered C32 to C10, L1 to L2, L3 to L4, MK2 to MK1, SW3 to SW1, SW1 to SW2, U1 to U3
Connections:
- net +3V3: now also J3.1 (Pin_1), C13.1, C14.1, C15.1, L13.2, L6.2, MK2.2 (SELECT), MK2.5 (VDD), R2.2, R21.2, R33.2, R50.2, R8.2, R9.2; no longer C26.1, C27.1, U3.2 (3V3)
- net DRV-HIZ_N: now also U3.17 (IO9); no longer U3.19 (IO11)
- net ESP-RXD: now also J3.5 (Pin_5)
- net ESP-TXD: now also J3.6 (Pin_6)
- net ESP_EN: now also R21.1
- net GIO48: now also J3.3 (Pin_3)
- net GND: now also IC2.2 (GND), MK1.2 (SELECT), C1.2, C12.2, C13.2, C14.2, C15.2, C19.2, C2.2, C20.2, C24.2, C28.2, C29.2, C4.2, C41.1, C44.2, C46.2, C5.2, C56.2, C57.2, C59.2, C6.2, C62.2, C7.2, C9.2, D1.A, IC1.2 (GND_1), IC1.4 (GND_2), IC5.2 (GND_1), IC5.4 (GND_2), J1.A1 (GND), J1.A12 (GND), J1.B1 (GND), J1.B12 (GND), J1.S1 (SHIELD), J9.14 (Pin_14), J9.9 (Pin_9), M11.1 (Pin_1), M12.1 (Pin_1), M13.1 (Pin_1), MK2.3_1 (GND), MK2.3_2 (GND), R12.1, R3.1, R52.1, R57.1, TP1.1, U1.13 (GND), U1.21 (PAD), U1.6 (RPD_G2), U1.7 (RPD_G1), U1.8 (GND), U2.11 (GND); no longer J3.1 (Pin_1)
- net HALL-A: now also U3.9 (IO16), C24.1
- net HALL-B: now also U3.10 (IO17), C28.1
- net HALL-C: now also U3.11 (IO18), C29.1
- net ISENS_A: now also R17.2
- net ISENS_B: now also R15.2
- net ISENS_C: now also R14.2
- net MIC_CLK: now also MK2.4 (CLOCK), R22.2; no longer U3.7 (IO7)
- net POT_SPEED: now also L8.1, R30.2; no longer U3.39 (IO1)
- net POT_TIME: now also L7.1, R32.2; no longer U3.38 (IO2)
- net SCL: now also R9.1, U2.7 (SCL); no longer J3.2 (Pin_2)
- net SDA: now also R8.1, U2.6 (SDA); no longer J3.3 (Pin_3)
- net VBUS: now also C56.1, IC5.3 (VIN), Q1.1 (S), Q1.2 (S), Q1.3 (S), Q5.5_6_7_8 (D), R51.1, R6.2
- net at IC2.1 (BOOT): now also C8.1
- net at IC2.3 (FB): now also R2.1, R3.2
- net at IC2.4 (EN): now also C3.1, IC2.5 (VIN), L2.2, C2.1
- net at IC2.6 (SW), L4.1: now also C8.2
- net at C21.1, U3.6 (IO6): now also R14.1
- net at C22.1, U3.5 (IO5): now also R15.1
- net at C23.1, U3.4 (IO4): now also R17.1
- net GIO46: now reaches U3.16 (IO46)
- net GIO46: now also J3.2 (Pin_2)
- net at U3.29 (IO36): now also R59.2
- net FAULT_RESET_IN: now reaches U3.30 (IO37)
- net FAULT_RESET_IN: now also L23.1
- net at U3.31 (IO38): now also R22.1
- net at U3.33 (IO40): now also C59.1, R50.1, R54.2
- net +BATT renamed +12V
- net +12V: now also C1.1, IC1.3 (VIN), Q1.5_6_7_8 (D), R11.2, R49.1, TP13.1
- net DRV-INHA renamed Motor Control/DRV-INHA
- net DRV-INHB renamed Motor Control/DRV-INHB
- net DRV-INHC renamed Motor Control/DRV-INHC
- net GIO21 renamed DRV_FAULT
- net GIO35: no longer names the net of U3.28 (IO35)
- net GIO35: now also R56.2
- net GIO39: no longer names the net of U3.32 (IO39)
- net GIO39: now also C44.1, R33.1, R53.2
- net GIO47 renamed SPEED_FAULT
- net MIC_DATA: no longer names the net of MK1.1 (DATA)
- net MIC_DATA: now also R7.2; no longer U3.12 (IO8)
- net POT_MIC: no longer names the net of U3.15 (IO3)
- net USB_N renamed USB_DM
- net USB_DM: now also U1.1 (C_SBU1), U2.3 (D-); no longer J3.6 (Pin_6)
- net USB_P renamed USB_DP
- net USB_DP: now also U1.2 (C_SBU2), U2.2 (D+); no longer J3.5 (Pin_5)
- net VBUS_SENSE renamed MIC_DATA2
- net MIC_DATA2: now also J9.16 (Pin_16); no longer C18.1
- net nFAULT: no longer names the net of U3.35 (IO42)
- net nFAULT: now also R61.2
- net nSLEEP: no longer names the net of U3.34 (IO41)
- net nSLEEP: now also R62.2
- new net: J9.3 (Pin_3), L8.2
- new net: C58.1, D9.1 (K), Q1.4 (G), R58.1
- new net: D9.2 (A), R5.2, R58.2, R6.1
- new net: C12.1, R51.2, U2.1 (VBUS)
- new net: R1.2, TP3.1
- new net: C26.1, C27.1, L13.1, U3.2 (3V3)
- new net: C62.1, Q5.4 (G), R72.1, R73.2
- new net: C41.2, U1.3 (VBIAS)
- new net: C19.1, J9.1 (Pin_1), L6.1
- new net: J9.4 (Pin_4), L9.2
- new net: J9.18 (Pin_18), L25.2
- new net: J1.A5 (CC1), U1.12 (CC1)
- new net: J1.A6 (D+), J1.B6 (D+), U1.14 (SBU2)
- new net: J1.A7 (D-), J1.B7 (D-), U1.15 (SBU1)
- new net: J1.B5 (CC2), U1.11 (CC2)
- new net: R5.1, U2.10 (GATE)
- new net: J9.2 (Pin_2), L7.2
- new net: J9.5 (Pin_5), L20.2
- new net: J9.6 (Pin_6), L21.2
- new net: J9.7 (Pin_7), L22.2
- new net: J9.8 (Pin_8), L23.2
- new net: U1.4 (C_CC1), U2.4 (CC1)
- new net: U1.5 (C_CC2), U2.5 (CC2)
- new net: R52.2, U2.8 (VSET)
- new net: R57.2, U2.9 (ISET)
- new net: C58.2, R49.2
- new net: MK2.1 (DATA), R10.2
- new net +5V: C6.1, C7.1, IC1.1 (VOUT)
- new net 3V3_LDO: C57.1, IC5.1 (VOUT), U1.10 (VPWR)
- new net 5V5: C20.1, J9.17 (Pin_17)
- new net MIC_CLK_BUFFERED: J9.15 (Pin_15), R55.1
- new net MIC_DATA1: R10.1, R7.1, U3.19 (IO11)
- new net Motor Control/MIC_CLOCK_BUFFERED: R55.2
- new net ON_BTN: L9.1, R73.1
- new net ON_LED_GB: J9.11 (Pin_11), R59.1
- new net ON_LED_R: J9.10 (Pin_10), R56.1
- new net PORT_FLT: R1.1, TP2.1, U1.9 (~{FLT})
- new net POT_SENSOR: L21.1, R60.2
- new net POT_SENS_FILT: C46.1, R60.1, U3.7 (IO7)
- new net POT_SPEED_FILT: C5.1, R30.1, U3.39 (IO1)
- new net POT_TIME_FILT: C9.1, R32.1, U3.38 (IO2)
- new net RESET_FAULT: L25.1
- new net SENSOR_BTN: L20.1, R54.1
- new net SENS_LED_GB: J9.13 (Pin_13), R61.1
- new net SENS_LED_R: J9.12 (Pin_12), R62.1
- new net START_BTN: L22.1, R53.1
- new net VBUS_CUT: C4.1, L3.2, Q5.1 (S), Q5.2 (S), Q5.3 (S), R72.2
- new net VBUS_PORT: F1.1, J1.A4 (VBUS), J1.A9 (VBUS), J1.B4 (VBUS), J1.B9 (VBUS)
- new net VBUS_TVS: D1.C, F1.2, L3.1
- new net VM_SENSE: C18.1, R11.1, R12.2, U3.12 (IO8)
- no-connect marks 12 -> 11
Other:
- added sheet Motor Control (motor_control.kicad_sch)
- added sheet interface_board (interface.kicad_sch)
- note removed: "switchable pullups (power saving during sleep)"
- company: Carlos Sabogal -> smoov dev ab
- title: project piCo 2 -> Sound activated motor driver
- moved on the sheet: C10, C11, C16, C18, C3, IC2, J3, J4, L2, L4, M1, M2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

Commit message: wip
Parts:
- removed C1, C2, C56, C57, C6, C7: 100NF 0402 25V X7R, smv_footprints:C_0402_1005Metric, symbol smv_capacitors:100NF 0402 25V X7R
- added C1, C56: 100NF_0603_100V_X7S, smv_footprints:C_0603_1608Metric, symbol smv_capacitors:100NF_0603_100V_X7S
- added C2: 10UF 1206 35V X5R, smv_footprints:C_1206_3216Metric, symbol smv_capacitors:10UF_1206_35V_X5R
- added C6, C7: 10UF_0805_16V_X7R, smv_footprints:C_0805_2012Metric, symbol smv_capacitors:10UF_0805_16V_X7R
- R55: value 10R 0402 -> 100R 0402; symbol smv_resistors:10R 0402 -> smv_resistors:100R 0402; val 10R -> 100R
Connections:
- net +12V: now also C56.1
- net +5V: now also C7.1
- net 3V3_LDO: now also C6.1
- net GND: now also C1.2, C2.2, C56.2, C6.2, C7.2
- net VBUS: now also C1.1
- net at C3.1, IC2.4 (EN), IC2.5 (VIN)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: now also C2.1
Other:
- moved on the sheet: C11, C15, MK1, MK2

Commit message: pre cleanup
Parts:
- J1: footprint Connector_USB:USB_C_Receptacle_GCT_USB4105-xx-A_16P_TopMnt_Horizontal -> (none)
- J9: value CONN_AMPHENOL_F51L-1A7H1-11018 -> JUSHUO AFA01-S18FCA-00; footprint smv_footprints:CONN_AMPHENOL_F51L-1A7H1-11018 -> smv_footprints:CONN_JUSHUO_JUSHUO AFA01-S18FCA-00; symbol smv_connectors_switches:CONN_AMPHENOL_F51L-1A7H1-11018 -> smv_connectors_switches:CONN_JUSHUO_AFA01-S18FCA-00; manf Amphenol ICC (FCI) -> JUSHUO; mpn F51L-1A7H1-11018 -> AFA01-S18FCA-00
- M1, M11, M12, M13, M2, M4, M5: footprint MountingHole:MountingHole_2.7mm_M2.5_ISO7380_Pad -> (none)
Connections:
- net VBUS: no longer IC5.3 (VIN)

Commit message: last data sent to jlc
Parts:
- removed J3: Conn_01x06_Pin, symbol Connector:Conn_01x06_Pin
- D1: MAXIMUM_PACKAGE_HEIGHT 0.6 mm -> (none); PARTREV 2 -> (none); STANDARD Manufacturer Recommendations -> (none)
- M1, M11, M12, M13, M2, M4, M5: footprint (none) -> MountingHole:MountingHole_2.7mm_M2.5_ISO7380_Pad
Connections:
- net VBUS: now also IC5.3 (VIN)
- net GIO46: no longer names the net of U3.16 (IO46)
- net GIO48: no longer names the net of U3.25 (IO48)
- net USB_DM renamed USB_N
- net USB_DP renamed USB_P
- no-connect marks 11 -> 13
