File: e003_source/interface.kicad_sch (KiCad schematic)
At the start: 34 parts, among them J2 CONN_AMPHENOL_F51L-1A7H1-11018, M10 CONN_M4_MOUNT, M3 CONN_M4_MOUNT, M6 CONN_M4_MOUNT, M7 CONN_M4_MOUNT, M8 CONN_M4_MOUNT, M9 CONN_M4_MOUNT

Commit message: last data sent to jlc
Parts:
- J2: value CONN_AMPHENOL_F51L-1A7H1-11018 -> JUSHUO AFA01-S18FCA-00; footprint smv_footprints:CONN_AMPHENOL_F51L-1A7H1-11018 -> smv_footprints:CONN_JUSHUO_JUSHUO AFA01-S18FCA-00; symbol smv_connectors_switches:CONN_AMPHENOL_F51L-1A7H1-11018 -> smv_connectors_switches:CONN_JUSHUO_AFA01-S18FCA-00; manf Amphenol ICC (FCI) -> JUSHUO; mpn F51L-1A7H1-11018 -> AFA01-S18FCA-00
