File: e003_source/motor_control.kicad_sch (KiCad schematic)
At the start: 76 parts, among them IC3 IC_TEXAS_NE556DR, IC4 DRV8317HREER, J5 B5P-VH, J6 CONN_JST_B6B-PH-K-S, K1 REL_PANASONIC_JW2SN-DC12V, Q2 TRAN_DIODES_DMN62D0U-13, Q3 TRAN_DIODES_DMN62D0U-13, Q4 TRAN_DIODES_DMN62D0U-13, Q6 TRAN_DIODES_DMN62D0U-13, U4 74HC393D, U5 IC_DIOD_LM4040D30FTA, U6 RS2254XQ, U7 IC_NEXPERIA_74LVC1G386GW, U8 74VHCT126AFT

Commit message: last data sent to jlc
Parts:
- IC3: Mouser Part Number 595-NE556DR -> (none); Mouser Price/Stock https://www.mouser.co.uk/ProductDetail/Texas-Instruments/NE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 -> (none)
